File: current-sensor.sch (KiCad schematic (older format))
At the start: 28 parts, among them J1 Molex_SL_01x02_Male, J2 Conn_01x04_Male, J3 Molex_SL_01x02_Male, SW1 SW_SP3T, SW2 SW_SP3T, U1 ACS730xLCTR-20AB, U2 AD8616xRM, U3 AD8616xRM, U4 LM1117-5.0

Commit message: fix opamp power unit annotation
Parts:
- renumbered U3 to U2, U4 to U3
Changed lines of the file:
@@
 TODO\n\nconsider different regulator\nbattery connector?\n\nregulator in/out caps:\nin: 10uF tant\nout: 10uF (ESR 0R3~~22R)
 $Comp
-L power:+5V #PWR?
+L power:+5V #PWR0102
 U 1 1 5EFBEFD8
 P 4200 1150
-F 0 "#PWR?" H 4200 1000 50  0001 C CNN
+F 0 "#PWR0102" H 4200 1000 50  0001 C CNN
 F 1 "+5V" H 4215 1323 50  0000 C CNN
 F 2 "" H 4200 1150 50  0001 C CNN
@@
 $EndComp
 $Comp
-L power:PWR_FLAG #FLG?
+L power:PWR_FLAG #FLG0101
 U 1 1 5EFBF412
 P 2400 1200
-F 0 "#FLG?" H 2400 1275 50  0001 C CNN
+F 0 "#FLG0101" H 2400 1275 50  0001 C CNN
 F 1 "PWR_FLAG" H 2400 1373 50  0000 C CNN
 F 2 "" H 2400 1200 50  0001 C CNN
@@
 	2400 1250 1350 1250
 $Comp
-L power:GND #PWR?
+L power:GND #PWR0103
 U 1 1 5EFC0FA6
 P 1450 1450
-F 0 "#PWR?" H 1450 1200 50  0001 C CNN
+F 0 "#PWR0103" H 1450 1200 50  0001 C CNN
 F 1 "GND" H 1455 1277 50  0000 C CNN
 F 2 "" H 1450 1450 50  0001 C CNN
@@
 	1450 1350 1350 1350
 $Comp
-L power:GND #PWR?
+L power:GND #PWR0104
 U 1 1 5EFC138B
 P 3350 1750
-F 0 "#PWR?" H 3350 1500 50  0001 C CNN
+F 0 "#PWR0104" H 3350 1500 50  0001 C CNN
 F 1 "GND" H 3355 1577 50  0000 C CNN
 F 2 "" H 3350 1750 50  0001 C CNN
@@
 $EndComp
 $Comp
-L power:GND #PWR?
+L power:GND #PWR0105
 U 1 1 5EFC981E
 P 3100 6450
-F 0 "#PWR?" H 3100 6200 50  0001 C CNN
+F 0 "#PWR0105" H 3100 6200 50  0001 C CNN
 F 1 "GND" H 3105 6277 50  0000 C CNN
 F 2 "" H 3100 6450 50  0001 C CNN
@@
 $EndComp
 $Comp
-L power:GND #PWR?
+L power:GND #PWR0106
 U 1 1 5EFCB33D
 P 3400 4050
-F 0 "#PWR?" H 3400 3800 50  0001 C CNN
+F 0 "#PWR0106" H 3400 3800 50  0001 C CNN
 F 1 "GND" H 3405 3877 50  0000 C CNN
 F 2 "" H 3400 4050 50  0001 C CNN
@@
 	2600 4000 2600 4050
 $Comp
-L power:+5V #PWR?
+L power:+5V #PWR0107
 U 1 1 5EFCC65B
 P 2600 3850
-F 0 "#PWR?" H 2600 3700 50  0001 C CNN
+F 0 "#PWR0107" H 2600 3700 50  0001 C CNN
 F 1 "+5V" H 2615 4023 50  0000 C CNN
 F 2 "" H 2600 3850 50  0001 C CNN
@@
 	5300 1450 5300 1600
 $Comp
-L power:GND #PWR?
+L power:GND #PWR0108
 U 1 1 5EFD9E68
 P 5300 2000
-F 0 "#PWR?" H 5300 1750 50  0001 C CNN
+F 0 "#PWR0108" H 5300 1750 50  0001 C CNN
 F 1 "GND" H 5305 1827 50  0000 C CNN
 F 2 "" H 5300 2000 50  0001 C CNN
@@
 	5300 2000 5300 1900
 $Comp
-L power:+5V #PWR?
+L power:+5V #PWR0109
 U 1 1 5EFDB3AC
 P 5300 1050
-F 0 "#PWR?" H 5300 900 50  0001 C CNN
+F 0 "#PWR0109" H 5300 900 50  0001 C CNN
 F 1 "+5V" H 5315 1223 50  0000 C CNN
 F 2 "" H 5300 1050 50  0001 C CNN
@@
 Connection ~ 5800 4450
 $Comp
-L Amplifier_Operational_gkeeth:AD8616xRM U3
+L Amplifier_Operational_gkeeth:AD8616xRM U2
 U 3 1 5F10C671
 P 5100 4450
-F 0 "U3" H 5158 4496 50  0001 L CNN
+F 0 "U2" H 5158 4496 50  0001 L CNN
 F 1 "AD8616xRM" H 5158 4405 50  0001 L CNN
 F 2 "Package_SO:MSOP-8_3x3mm_P0.65mm" H 5200 4450 50  0001 C CNN
@@
 $EndComp
 $Comp
-L Amplifier_Operational_gkeeth:AD8616xRM U4
+L Amplifier_Operational_gkeeth:AD8616xRM U3
 U 3 1 5F10CA04
 P 4200 5950
-F 0 "U4" H 4258 5996 50  0001 L CNN
+F 0 "U3" H 4258 5996 50  0001 L CNN
 F 1 "AD8616xRM" H 4258 5905 50  0001 L CNN
 F 2 "Package_SO:MSOP-8_3x3mm_P0.65mm" H 4300 5950 50  0001 C CNN
@@
 $EndComp
 $Comp
-L power:GND #PWR?
+L power:GND #PWR0110
 U 1 1 5F1117EC
 P 4200 6300
-F 0 "#PWR?" H 4200 6050 50  0001 C CNN
+F 0 "#PWR0110" H 4200 6050 50  0001 C CNN
 F 1 "GND" H 4205 6127 50  0000 C CNN
 F 2 "" H 4200 6300 50  0001 C CNN
@@
 	4200 6300 4200 6250
 $Comp
-L power:+5V #PWR?
+L power:+5V #PWR0111
 U 1 1 5F117ABF
 P 4200 5450
-F 0 "#PWR?" H 4200 5300 50  0001 C CNN
+F 0 "#PWR0111" H 4200 5300 50  0001 C CNN
 F 1 "+5V" H 4215 5623 50  0000 C CNN
 F 2 "" H 4200 5450 50  0001 C CNN
@@
 	4200 5550 4200 5450
 $Comp
-L power:GND #PWR?
+L power:GND #PWR0112
 U 1 1 5F11EE97
 P 3850 5600
-F 0 "#PWR?" H 3850 5350 50  0001 C CNN
+F 0 "#PWR0112" H 3850 5350 50  0001 C CNN
 F 1 "GND" H 3855 5427 50  0000 C CNN
 F 2 "" H 3850 5600 50  0001 C CNN
@@
 	3850 5550 3900 5550
 $Comp
-L power:+5V #PWR?
+L power:+5V #PWR0113
 U 1 1 5F124EA8
 P 5100 3950
-F 0 "#PWR?" H 5100 3800 50  0001 C CNN
+F 0 "#PWR0113" H 5100 3800 50  0001 C CNN
 F 1 "+5V" H 5115 4123 50  0000 C CNN
 F 2 "" H 5100 3950 50  0001 C CNN
@@
 	5100 4050 5100 3950
 $Comp
-L power:GND #PWR?
+L power:GND #PWR0114
 U 1 1 5F124EB8
 P 4750 4100
-F 0 "#PWR?" H 4750 3850 50  0001 C CNN
+F 0 "#PWR0114" H 4750 3850 50  0001 C CNN
 F 1 "GND" H 4755 3927 50  0000 C CNN
 F 2 "" H 4750 4100 50  0001 C CNN
@@
 	4750 4050 4800 4050
 $Comp
-L power:GND #PWR?
+L power:GND #PWR0115
 U 1 1 5F13C796
 P 5100 4800
-F 0 "#PWR?" H 5100 4550 50  0001 C CNN
+F 0 "#PWR0115" H 5100 4550 50  0001 C CNN
 F 1 "GND" H 5105 4627 50  0000 C CNN
 F 2 "" H 5100 4800 50  0001 C CNN

Commit message: mostly complete schematic and initial placement
Parts:
- removed D1: LED, symbol Device:LED
- removed J2: Conn_01x04_Male, Connector_Molex_KK-396:Molex_KK-396_A-41791-0004_1x04_P3.96mm_Vertical, symbol Connector:Conn_01x04_Male
- removed J3: Molex_SL_01x02_Male, Connector_Molex_SL:Molex_SL_A-70543-0001_1x02_P2.54mm_Vertical, symbol Connector_gkeeth:Molex_SL_01x02_Male
- removed SW1, SW2: SW_SP3T, symbol Switch:SW_SP3T
- removed U1: ACS730xLCTR-20AB, Package_SO:SOIC-8_3.9x4.9mm_P1.27mm, symbol Sensor_Current:ACS730xLCTR-20AB
- removed U4: LM1117-5.0, Package_TO_SOT_SMD:SOT-223-3_TabPin2, symbol Regulator_Linear:LM1117-5.0
- added H1, H2, H3, H4: MountingHole, MountingHole:MountingHole_3.2mm_M3, symbol Mechanical:MountingHole
- added J1, J2: ‎0197134001‎, Connector_Molex_Quixon:Connector_Molex_Quixon_19713-4001_1x01_Horizontal, symbol Connector:Conn_01x01_Male
- added J3: 0731000105, Connector_Coaxial_gkeeth:BNC_Molex_73100-0105_Horizontal, symbol Connector:Conn_Coaxial
- added J5: Molex_SL_01x02_Male, Connector_Molex_SL:Molex_SL_A-70543-0001_1x02_P2.54mm_Vertical, symbol Connector_gkeeth:Molex_SL_01x02_Male
- added SW1: PN12Sxxx03QE, Button_Switch_THT_gkeeth:SW_Push_SPDT_CK_PN1xSxxx03QE, symbol Switch_gkeeth:PN12Sxxx03QE
- added SW2, SW3: OS103011MA7QP1, Button_Switch_THT_gkeeth:SW_Slide_SP3T_CK_OS103011MA7QP1, symbol Switch_gkeeth:OS103011MA7QP1
- added U1: ACS730xLCTR-20AB, Package_SO:SOIC-8_3.9x4.9mm_P1.27mm, symbol Sensor_Current_gkeeth:ACS730xLCTR-20AB
- added U4: NCP718ASN500, Package_TO_SOT_SMD:TSOT-23-5, symbol Regulator_Linear_gkeeth:NCP718ASN500
- C1, C2, C3, C4, C5, C6, C7: footprint (none) -> Capacitor_SMD:C_0603_1608Metric
- C8, C9: value C -> 1u; footprint (none) -> Capacitor_SMD:C_0603_1608Metric
- R1, R2, R3, R4, R5, R6, R7, R8: footprint (none) -> Resistor_SMD:R_0603_1608Metric
- renumbered J1 to J4
Connections:
- wire segments 116 -> 115
- no-connect marks 0 -> 2
Other:
- note added: "TODO\ncheck power switch pinout\nchange power switch PN to actually ordered one\nmake holes the right size"
- note added: "To banana jacks"
- note added: "to 9V battery"
- note added: "to front-panel power LED"
- note removed: "TODO\n\nconsider different regulator\nbattery connector?\n\nregulator in/out caps:\nin: 10uF tant\nout: 10uF (ESR 0R3~~22R)"
- note removed: "To BNC"
- note removed: "To bananas"
- moved on the sheet: C8, J4, R8

Commit message: add mechanical models for enclosure, battery holder, and binding posts
Other:
- note added: "#4 clearance hole is approx. 3.2mm (M3)"
Changed lines of the file:
@@
 Text Notes 2400 1450 0    50   ~ 10
 to 9V battery
+Text Notes 950  8000 0    50   ~ 0
+#4 clearance hole is approx. 3.2mm (M3)
 $EndSCHEMATC

Commit message: complete mechanical placement of all components on main pcb, and holes on front/back panels
Parts:
- added LOGO2: Logo_MadeWithKiCad, Symbol:KiCad-Logo2_6mm_SilkScreen, symbol Graphic_gkeeth:Logo_MadeWithKiCad
- added LOGO3: Logo_Open_Hardware_Small, Symbol:OSHW-Logo2_7.3x6mm_SilkScreen, symbol Graphic:Logo_Open_Hardware_Small
- U1: value ACS730xLCTR-20AB -> ACS730xLCTR-40AB; symbol Sensor_Current_gkeeth:ACS730xLCTR-20AB -> Sensor_Current_gkeeth:ACS730xLCTR-40AB
Changed lines of the file:
@@
 L Creative_Commons:CC-BY-SA_0.5in LOGO1
 U 1 1 5EFB5A29
-P 5150 7400
-F 0 "LOGO1" H 5150 7180 60  0001 C CNN
-F 1 "CC-BY-SA_0.5in" H 5150 7620 60  0001 C CNN
-F 2 "Symbol_CreativeCommons:CC-BY-SA_SilkScreenTop_Small" H 5150 7400 50  0001 C CNN
-F 3 "" H 5150 7400 50  0001 C CNN
-	1    5150 7400
+P 5000 7050
+F 0 "LOGO1" H 5000 6830 60  0001 C CNN
+F 1 "CC-BY-SA_0.5in" H 5000 7270 60  0001 C CNN
+F 2 "Symbol_CreativeCommons:CC-BY-SA_SilkScreenTop_Small" H 5000 7050 50  0001 C CNN
+F 3 "" H 5000 7050 50  0001 C CNN
+	1    5000 7050
 	1    0    0    -1
 $EndComp
@@
 $EndComp
 $Comp
-L Sensor_Current_gkeeth:ACS730xLCTR-20AB U1
+L Sensor_Current_gkeeth:ACS730xLCTR-40AB U1
 U 1 1 5F083F8B
 P 2600 4350
 F 0 "U1" H 2850 4600 50  0000 C CNN
-F 1 "ACS730xLCTR-20AB" H 2100 4600 50  0000 C CNN
+F 1 "ACS730xLCTR-40AB" H 2100 4600 50  0000 C CNN
 F 2 "Package_SO:SOIC-8_3.9x4.9mm_P1.27mm" H 2950 4250 50  0001 L CIN
 F 3 "http://www.allegromicro.com/~/media/Files/Datasheets/ACS730-Datasheet.ashx?la=en" H 2600 4350 50  0001 C CNN
@@
 Text Notes 950  8000 0    50   ~ 0
 #4 clearance hole is approx. 3.2mm (M3)
+$Comp
+L Graphic_gkeeth:Logo_MadeWithKiCad LOGO2
+U 1 1 5F364A72
+P 4600 7750
+F 0 "LOGO2" H 4600 7750 50  0001 C CNN
+F 1 "Logo_MadeWithKiCad" H 4600 7750 50  0001 C CNN
+F 2 "Symbol:KiCad-Logo2_6mm_SilkScreen" H 4600 7750 50  0001 C CNN
+F 3 "" H 4600 7750 50  0001 C CNN
+	1    4600 7750
+	1    0    0    -1
+$EndComp
+$Comp
+L Graphic:Logo_Open_Hardware_Small LOGO3
+U 1 1 5F365262
+P 5750 7700
+F 0 "LOGO3" H 5750 7975 50  0001 C CNN
+F 1 "Logo_Open_Hardware_Small" H 5750 7475 50  0001 C CNN
+F 2 "Symbol:OSHW-Logo2_7.3x6mm_SilkScreen" H 5750 7700 50  0001 C CNN
+F 3 "~" H 5750 7700 50  0001 C CNN
+	1    5750 7700
+	1    0    0    -1
+$EndComp
 $EndSCHEMATC
