File: current-sensor-frontpanel/current-sensor-frontpanel.kicad_pcb (KiCad board)
At the start: 2 copper layers, 98 x 30 mm, 9 parts

Commit message: generate gerbers for 36A and 20A frontpanel
Other:
- board text added: "Current Sensor Front Panel r0 G. Keeth github.com/gkeeth/current-sensor 2020-10-25"
- board text removed: "Current Sensor Front Panel r0 G. Keeth github.com/gkeeth/current-sensor 2020-10-23"
